Commit message: [add] create simulation environment

File: resources/sciurus17/sciurus17.urdf (robot description, URDF)
Before this commit: robot sciurus17, 26 links, 25 joints
Links:
- link base_link: geometry collision mesh filename=meshes/collision/Base.stl scale=1.0 1.0 1.0; visual mesh filename=meshes/visual/Base.stl scale=1.0 1.0 1.0
- link body_link: geometry collision mesh filename=meshes/collision/Body.stl scale=1.0 1.0 1.0; visual mesh filename=meshes/visual/Body.stl scale=1.0 1.0 1.0
- link l_handA_link: geometry collision mesh filename=meshes/collision/L_HandA.stl scale=1.0 1.0 1.0; visual mesh filename=meshes/visual/L_HandA.stl scale=1.0 1.0 1.0
- link l_handB_link: geometry collision mesh filename=meshes/collision/L_HandB.stl scale=1.0 1.0 1.0; visual mesh filename=meshes/visual/L_HandB.stl scale=1.0 1.0 1.0
- link l_link1: geometry collision mesh filename=meshes/collision/L_Link1.stl scale=1.0 1.0 1.0; visual mesh filename=meshes/visual/L_Link1.stl scale=1.0 1.0 1.0
- link l_link2: geometry collision mesh filename=meshes/collision/L_Link2.stl scale=-1.0 1.0 -1.0; visual mesh filename=meshes/visual/L_Link2.stl scale=-1.0 1.0 -1.0
- link l_link3: geometry collision mesh filename=meshes/collision/L_Link3.stl scale=1.0 1.0 1.0; visual mesh filename=meshes/visual/L_Link3.stl scale=1.0 1.0 1.0
- link l_link4: geometry collision mesh filename=meshes/collision/L_Link4.stl scale=1.0 1.0 1.0; visual mesh filename=meshes/visual/L_Link4.stl scale=1.0 1.0 1.0
- link l_link5: geometry collision mesh filename=meshes/collision/L_Link5.stl scale=1.0 1.0 1.0; visual mesh filename=meshes/visual/L_Link5.stl scale=1.0 1.0 1.0
- link l_link6: geometry collision mesh filename=meshes/collision/L_Link6.stl scale=1.0 1.0 1.0; visual mesh filename=meshes/visual/L_Link6.stl scale=1.0 1.0 1.0
- link l_link7: geometry collision mesh filename=meshes/collision/L_Link7.stl scale=1.0 1.0 1.0; visual mesh filename=meshes/visual/L_Link7.stl scale=1.0 1.0 1.0
- link neck_pitch_link: geometry collision mesh filename=meshes/collision/Neck2.stl scale=1.0 1.0 1.0; visual mesh filename=meshes/visual/Neck2.stl scale=1.0 1.0 1.0
- link neck_yaw_link: geometry collision mesh filename=meshes/collision/Neck1.stl scale=1.0 1.0 1.0; visual mesh filename=meshes/visual/Neck1.stl scale=1.0 1.0 1.0
- link r_handA_link: geometry collision mesh filename=meshes/collision/R_HandA.stl scale=1.0 1.0 1.0; visual mesh filename=meshes/visual/R_HandA.stl scale=1.0 1.0 1.0
- link r_handB_link: geometry collision mesh filename=meshes/collision/R_HandB.stl scale=1.0 1.0 1.0; visual mesh filename=meshes/visual/R_HandB.stl scale=1.0 1.0 1.0
- link r_link1: geometry collision mesh filename=meshes/collision/R_Link1.stl scale=1.0 1.0 1.0; visual mesh filename=meshes/visual/R_Link1.stl scale=1.0 1.0 1.0
- link r_link2: geometry collision mesh filename=meshes/collision/R_Link2.stl scale=1.0 1.0 1.0; visual mesh filename=meshes/visual/R_Link2.stl scale=1.0 1.0 1.0
- link r_link3: geometry collision mesh filename=meshes/collision/L_Link3.stl scale=1.0 -1.0 1.0; visual mesh filename=meshes/visual/L_Link3.stl scale=1.0 -1.0 1.0
- link r_link4: geometry collision mesh filename=meshes/collision/R_Link4.stl scale=1.0 1.0 1.0; visual mesh filename=meshes/visual/R_Link4.stl scale=1.0 1.0 1.0
- link r_link5: geometry collision mesh filename=meshes/collision/R_Link5.stl scale=1.0 1.0 1.0; visual mesh filename=meshes/visual/Logo_Corp.stl scale=1.0 1.0 1.0
- link r_link6: geometry collision mesh filename=meshes/collision/R_Link6.stl scale=1.0 1.0 1.0; visual mesh filename=meshes/visual/R_Link6.stl scale=1.0 1.0 1.0
- link r_link7: geometry collision mesh filename=meshes/collision/R_Link7.stl scale=1.0 1.0 1.0; visual mesh filename=meshes/visual/R_Link7.stl scale=1.0 1.0 1.0
